File: LED_MATRIX.kicad_sch (KiCad schematic)
At the start: 16 parts, among them U1 AS1115-BSST, U2 ESP32-S3-WROOM-1

Commit message: wip
Parts:
- removed D13, D14: LED, symbol Device:LED
- removed U2: ESP32-S3-WROOM-1, RF_Module:ESP32-S3-WROOM-1, symbol RF_Module:ESP32-S3-WROOM-1
- added J1, J2, J3: Conn_01x01, symbol Connector_Generic:Conn_01x01
- added R1: 9.53kOhm, symbol Device:R
Connections:
- net at D10.1 (K), D8.1 (K), D9.1 (K): now also D6.1 (K), D7.1 (K), U1.2 (DIG0); no longer D11.1 (K), D12.1 (K), U1.3 (DIG1)
- net at D4.2 (A), U1.23 (SEGD): now also D9.2 (A); no longer D11.2 (A)
- net at D1.1 (K), D2.1 (K), D3.1 (K)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: now also U1.3 (DIG1); no longer D6.1 (K), D7.1 (K), U1.2 (DIG0)
- net at D10.2 (A), U1.21 (SEGE): now also D12.2 (A), D5.2 (A); no longer D3.2 (A)
- net at U1.15 (SEGA): now also D1.2 (A), D11.2 (A), D6.2 (A); no longer D7.2 (A)
- net at U1.17 (SEGB): now also D2.2 (A), D7.2 (A); no longer D6.2 (A)
- net at U1.1 (SDA): now also J2.1 (Pin_1)
- net at U1.13 (ISET): now also R1.2
- net at U1.14 (SCL): now also J1.1 (Pin_1)
- net at U1.24 (IRQ): now also J3.1 (Pin_1)
- net at U1.4 (DIG2): now also D11.1 (K), D12.1 (K)
- new net: D3.2 (A), D8.2 (A), U1.20 (SEGC)
- new net +5V: R1.1
- now unconnected: U1.16 (SEGF), U1.18 (SEGG)
- no-connect marks 0 -> 10

Commit message: wip
Parts:
- removed J3: Conn_01x01, symbol Connector_Generic:Conn_01x01
Connections:
- net +5V is gone; now on net VCC: R1.1
- no-connect marks 10 -> 11
Changed lines of the file:
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@@
+	)
+	(no_connect
+		(at 140.97 63.5)
 	)
 	(no_connect
@@
 	(wire
 		(pts
-			(xy 140.97 67.31) (xy 130.81 67.31)
-		)
-		(stroke
-			(width 0)
-			(type default)
-		)
-	)
-	(wire
-		(pts
 			(xy 187.96 22.86) (xy 184.15 22.86)
 		)
@@
 		(pts
 			(xy 171.45 68.58) (xy 189.23 68.58)
-		)
-		(stroke
-			(width 0)
-			(type default)
-		)
-	)
-	(wire
-		(pts
-			(xy 140.97 63.5) (xy 140.97 67.31)
 		)
 		(stroke
@@
 	)
 	(symbol
-		(lib_id "Connector_Generic:Conn_01x01")
-		(at 125.73 67.31 180)
-		(unit 1)
-		(exclude_from_sim no)
-		(in_bom yes)
-		(on_board yes)
-		(dnp no)
-		(property "Reference" "J3"
-			(at 122.682 67.31 0)
-			(effects
-				(font
-					(size 1.27 1.27)
-				)
-			)
-		)
-		(property "Value" "Conn_01x01"
-			(at 125.73 69.85 0)
-			(effects
-				(font
-					(size 1.27 1.27)
-				)
-			)
-		)
-		(property "Footprint" ""
-			(at 125.73 67.31 0)
-			(effects
-				(font
-					(size 1.27 1.27)
-				)
-				(hide yes)
-			)
-		)
-		(property "Datasheet" "~"
-			(at 125.73 67.31 0)
-			(effects
-				(font
-					(size 1.27 1.27)
-				)
-				(hide yes)
-			)
-		)
-		(property "Description" "Generic connector, single row, 01x01, script generated (kicad-library-utils/schlib/autogen/connector/)"
-			(at 125.73 67.31 0)
-			(effects
-				(font
-					(size 1.27 1.27)
-				)
-				(hide yes)
-			)
-		)
-		(pin "1"
-		)
-		(instances
-			(project ""
-				(path "/3e9d6c2e-f289-4b1b-ad37-c26dbc105080"
-					(reference "J3")
-					(unit 1)
-				)
-			)
-		)
-	)
-	(symbol
 		(lib_id "Device:LED")
 		(at 217.17 29.21 90)
@@
 				(path "/3e9d6c2e-f289-4b1b-ad37-c26dbc105080"
 					(reference "D7")
+					(unit 1)
+				)
+			)
+		)
+	)
+	(symbol
+		(lib_id "power:VCC")
+		(at 123.19 44.45 90)
+		(unit 1)
+		(exclude_from_sim no)
+		(in_bom yes)
+		(on_board yes)
+		(dnp no)
+		(fields_autoplaced yes)
+		(property "Reference" "#PWR01"
+			(at 127 44.45 0)
+			(effects
+				(font
+					(size 1.27 1.27)
+				)
+				(hide yes)
+			)
+		)
+		(property "Value" "VCC"
+			(at 119.38 44.4499 90)
+			(effects
+				(font
+					(size 1.27 1.27)
+				)
+				(justify left)
+			)
+		)
+		(property "Footprint" ""
+			(at 123.19 44.45 0)
+			(effects
+				(font
+					(size 1.27 1.27)
+				)
+				(hide yes)
+			)
+		)
+		(property "Datasheet" ""
+			(at 123.19 44.45 0)
+			(effects
+				(font
+					(size 1.27 1.27)
+				)
+				(hide yes)
+			)
+		)
+		(property "Description" "Power symbol creates a global label with name \"VCC\""
+			(at 123.19 44.45 0)
+			(effects
+				(font
+					(size 1.27 1.27)
+				)
+				(hide yes)
+			)
+		)
+		(pin "1"
+		)
+		(instances
+			(project "LED_MATRIX"
+				(path "/3e9d6c2e-f289-4b1b-ad37-c26dbc105080"
+					(reference "#PWR01")
 					(unit 1)
 				)
@@
 					(unit 1)
 				)
-			)
-		)
-	)
-	(symbol
-		(lib_id "power:+5V")
-		(at 123.19 44.45 90)
-		(unit 1)
-		(exclude_from_sim no)
-		(in_bom yes)
-		(on_board yes)
-		(dnp no)
-		(fields_autoplaced yes)
-		(property "Reference" "#PWR01"
-			(at 127 44.45 0)
-			(effects
-				(font
-					(size 1.27 1.27)
-				)
-				(hide yes)
-			)
-		)
-		(property "Value" "+5V"
-			(at 119.38 44.4499 90)
-			(effects
-				(font
-					(size 1.27 1.27)
-				)
-				(justify left)
-			)
-		)
-		(property "Footprint" ""
-			(at 123.19 44.45 0)
-			(effects
-				(font
-					(size 1.27 1.27)
-				)
-				(hide yes)
-			)
-		)
-		(property "Datasheet" ""
-			(at 123.19 44.45 0)
-			(effects
-				(font
-					(size 1.27 1.27)
-				)
-				(hide yes)
-			)
-		)
-		(property "Description" "Power symbol creates a global label with name \"+5V\""
-			(at 123.19 44.45 0)
-			(effects
-				(font
-					(size 1.27 1.27)
-				)
-				(hide yes)
-			)
-		)
-		(pin "1"
-		)
-		(instances
-			(project ""
-				(path "/3e9d6c2e-f289-4b1b-ad37-c26dbc105080"
-					(reference "#PWR01")
-					(unit 1)
-				)

Commit message: wip
Parts:
- D1, D10, D11, D12, D2, D3, D4, D5, D6, D7, D8, D9: footprint (none) -> Footprints:Bivar_1206_SMD
- J1, J2: footprint (none) -> TestPoint:TestPoint_Pad_2.5x2.5mm
- R1: footprint (none) -> Resistor_THT:R_Axial_DIN0204_L3.6mm_D1.6mm_P2.54mm_Vertical
Changed lines of the file:
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@@
 			)
 		)
-		(property "Footprint" ""
+		(property "Footprint" "Footprints:Bivar_1206_SMD"
 			(at 204.47 74.93 0)
 			(effects
@@
 			)
 		)
-		(property "Footprint" ""
+		(property "Footprint" "Footprints:Bivar_1206_SMD"
 			(at 217.17 29.21 0)
 			(effects
@@
 			)
 		)
-		(property "Footprint" ""
+		(property "Footprint" "Footprints:Bivar_1206_SMD"
 			(at 217.17 74.93 0)
 			(effects
@@
 			)
 		)
-		(property "Footprint" ""
+		(property "Footprint" "Footprints:Bivar_1206_SMD"
 			(at 187.96 29.21 0)
 			(effects
@@
 			)
 		)
-		(property "Footprint" ""
+		(property "Footprint" "Footprints:Bivar_1206_SMD"
 			(at 208.28 59.69 0)
 			(effects
@@
 			)
 		)
-		(property "Footprint" ""
+		(property "Footprint" "Footprints:Bivar_1206_SMD"
 			(at 198.12 74.93 0)
 			(effects
@@
 			)
 		)
-		(property "Footprint" ""
+		(property "Footprint" "Footprints:Bivar_1206_SMD"
 			(at 201.93 59.69 0)
 			(effects
@@
 			)
 		)
-		(property "Footprint" ""
+		(property "Footprint" "Footprints:Bivar_1206_SMD"
 			(at 210.82 74.93 0)
 			(effects
@@
 			)
 		)
-		(property "Footprint" ""
+		(property "Footprint" "Footprints:Bivar_1206_SMD"
 			(at 191.77 74.93 0)
 			(effects
@@
 			)
 		)
-		(property "Footprint" ""
+		(property "Footprint" "Footprints:Bivar_1206_SMD"
 			(at 195.58 59.69 0)
 			(effects
@@
 			)
 		)
-		(property "Footprint" ""
+		(property "Footprint" "TestPoint:TestPoint_Pad_2.5x2.5mm"
 			(at 125.73 54.61 0)
 			(effects
@@
 			)
 		)
-		(property "Footprint" ""
+		(property "Footprint" "TestPoint:TestPoint_Pad_2.5x2.5mm"
 			(at 125.73 60.96 0)
 			(effects
@@
 			)
 		)
-		(property "Footprint" ""
+		(property "Footprint" "Footprints:Bivar_1206_SMD"
 			(at 214.63 59.69 0)
 			(effects
@@
 			)
 		)
-		(property "Footprint" ""
+		(property "Footprint" "Footprints:Bivar_1206_SMD"
 			(at 189.23 59.69 0)
 			(effects
@@
 			)
 		)
-		(property "Footprint" ""
+		(property "Footprint" "Resistor_THT:R_Axial_DIN0204_L3.6mm_D1.6mm_P2.54mm_Vertical"
 			(at 127 46.228 90)
 			(effects

Commit message: wip
Parts:
- R1: footprint Resistor_THT:R_Axial_DIN0204_L3.6mm_D1.6mm_P2.54mm_Vertical -> Resistor_SMD:R_0201_0603Metric
Changed lines of the file:
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@@
 			)
 		)
-		(property "Footprint" "Resistor_THT:R_Axial_DIN0204_L3.6mm_D1.6mm_P2.54mm_Vertical"
+		(property "Footprint" "Resistor_SMD:R_0201_0603Metric"
 			(at 127 46.228 90)
 			(effects

Commit message: wip
Parts:
- J1, J2: footprint TestPoint:TestPoint_Pad_2.5x2.5mm -> TestPoint:TestPoint_THTPad_2.0x2.0mm_Drill1.0mm
- R1: footprint Resistor_SMD:R_0201_0603Metric -> Resistor_SMD:R_0805_2012Metric_Pad1.20x1.40mm_HandSolder
Changed lines of the file:
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@@
 			)
 		)
-		(property "Footprint" "TestPoint:TestPoint_Pad_2.5x2.5mm"
+		(property "Footprint" "TestPoint:TestPoint_THTPad_2.0x2.0mm_Drill1.0mm"
 			(at 125.73 54.61 0)
 			(effects
@@
 			)
 		)
-		(property "Footprint" "TestPoint:TestPoint_Pad_2.5x2.5mm"
+		(property "Footprint" "TestPoint:TestPoint_THTPad_2.0x2.0mm_Drill1.0mm"
 			(at 125.73 60.96 0)
 			(effects
@@
 			)
 		)
-		(property "Footprint" "Resistor_SMD:R_0201_0603Metric"
+		(property "Footprint" "Resistor_SMD:R_0805_2012Metric_Pad1.20x1.40mm_HandSolder"
 			(at 127 46.228 90)
 			(effects

Commit message: wip
Parts:
- added U2: TLC5940PWP, Package_SO:HTSSOP-28-1EP_4.4x9.7mm_P0.65mm_EP3.4x9.5mm_Mask2.4x6.17mm_ThermalVias, symbol Driver_LED:TLC5940PWP
Changed lines of the file:
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@@
+	)
+	(symbol
+		(lib_id "Driver_LED:TLC5940PWP")
+		(at 99.06 96.52 0)
+		(unit 1)
+		(exclude_from_sim no)
+		(in_bom yes)
+		(on_board yes)
+		(dnp no)
+		(fields_autoplaced yes)
+		(property "Reference" "U2"
+			(at 101.2033 71.12 0)
+			(effects
+				(font
+					(size 1.27 1.27)
+				)
+				(justify left)
+			)
+		)
+		(property "Value" "TLC5940PWP"
+			(at 101.2033 73.66 0)
+			(effects
+				(font
+					(size 1.27 1.27)
+				)
+				(justify left)
+			)
+		)
+		(property "Footprint" "Package_SO:HTSSOP-28-1EP_4.4x9.7mm_P0.65mm_EP3.4x9.5mm_Mask2.4x6.17mm_ThermalVias"
+			(at 99.695 121.285 0)
+			(effects
+				(font
+					(size 1.27 1.27)
+				)
+				(justify left)
+				(hide yes)
+			)
+		)
+		(property "Datasheet" "http://www.ti.com/lit/ds/symlink/tlc5940.pdf"
+			(at 88.9 78.74 0)
+			(effects
+				(font
+					(size 1.27 1.27)
+				)
+				(hide yes)
+			)
+		)
+		(property "Description" "16-Channel LED Driver With DOT Correction and Grayscale PWM Control, TSSOP package with thermal pad"
+			(at 99.06 96.52 0)
+			(effects
+				(font
+					(size 1.27 1.27)
+				)
+				(hide yes)
+			)
+		)
+		(pin "8"
+		)
+		(pin "17"
+		)
+		(pin "12"
+		)
+		(pin "1"
+		)
+		(pin "4"
+		)
+		(pin "23"
+		)
+		(pin "3"
+		)
+		(pin "25"
+		)
+		(pin "26"
+		)
+		(pin "5"
+		)
+		(pin "27"
+		)
+		(pin "6"
+		)
+		(pin "14"
+		)
+		(pin "2"
+		)
+		(pin "29"
+		)
+		(pin "20"
+		)
+		(pin "15"
+		)
+		(pin "19"
+		)
+		(pin "16"
+		)
+		(pin "13"
+		)
+		(pin "9"
+		)
+		(pin "11"
+		)
+		(pin "7"
+		)
+		(pin "21"
+		)
+		(pin "22"
+		)
+		(pin "24"
+		)
+		(pin "18"
+		)
+		(pin "28"
+		)
+		(pin "10"
+		)
+		(instances
+			(project ""
+				(path "/3e9d6c2e-f289-4b1b-ad37-c26dbc105080"
+					(reference "U2")
+					(unit 1)
+				)
+			)
+		)
 	)
 	(symbol

Commit message: wip
Parts:
- removed J1, J2: Conn_01x01, TestPoint:TestPoint_THTPad_2.0x2.0mm_Drill1.0mm, symbol Connector_Generic:Conn_01x01
- removed R1: 9.53kOhm, Resistor_SMD:R_0805_2012Metric_Pad1.20x1.40mm_HandSolder, symbol Device:R
- removed U1: AS1115-BSST, Package_SO:QSOP-24_3.9x8.7mm_P0.635mm, symbol Interface_Expansion:AS1115-BSST
Connections:
- net VCC: now also D1.2 (A), D10.2 (A), D11.2 (A), D12.2 (A), D2.2 (A), D3.2 (A), D4.2 (A), D5.2 (A), D6.2 (A), D7.2 (A), D8.2 (A), D9.2 (A)
- net at D12.1 (K): no longer D11.1 (K)
- net at U2.20 (OUT13): now also D3.1 (K)
- net at U2.21 (OUT14): now also D2.1 (K)
- net at U2.22 (OUT15): now also D1.1 (K)
- now unconnected: D10.1 (K), D4.1 (K), D5.1 (K), D6.1 (K), D7.1 (K), D8.1 (K), D9.1 (K)
- no-connect marks 11 -> 0
Other:
- moved on the sheet: D1, D10, D11, D12, D2, D3, D4, D5, D6, D7, D8, D9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

Commit message: wip
Parts:
- added TP1, TP2, TP3, TP4, TP5: TestPoint, TestPoint:TestPoint_Pad_1.5x1.5mm, symbol Connector:TestPoint
Connections:
- net VCC: now also U2.26 (DCPRG), U2.28 (VCC)
- net at D8.1 (K): now also U2.15 (OUT8)
- net at D12.1 (K): now also U2.11 (OUT4)
- net at D10.1 (K): now also U2.13 (OUT6)
- net at D11.1 (K): now also U2.12 (OUT5)
- net at D4.1 (K): now also U2.19 (OUT12)
- net at D7.1 (K): now also U2.16 (OUT9)
- net at D9.1 (K): now also U2.14 (OUT7)
- net at D6.1 (K): now also U2.17 (OUT10)
- net at D5.1 (K): now also U2.18 (OUT11)
- net GND: now reaches U2.1 (GND)
- net GND: now also U2.6 (VPRG)
- net at U2.2 (BLANK): now also TP2.1
- net at U2.25 (GSCLK): now also TP5.1
- net at U2.3 (XLAT): now also TP4.1
- net at U2.4 (SCLK): now also TP1.1
- net at U2.5 (SIN): now also TP3.1
- no-connect marks 0 -> 6
Other:
- company: (none) -> HAW Hamburg
- title: (none) -> Led Matrix
- moved on the sheet: D1, D10, D11, D12, D2, D3, D4, D5, D6, D7, D8, D9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
