File: LED_MATRIX.kicad_sch (KiCad schematic)
At the start: 18 parts, among them U2 TLC5940PWP

Commit message: wip
Parts:
- added R1: 2kO, symbol Device:R
Connections:
- net GND: now also R1.1
- net at U2.27 (IREF): now also R1.2
Changed lines of the file:
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@@
+	)
+	(junction
+		(at 149.86 96.52)
+		(diameter 0)
+		(color 0 0 0 0)
 	)
 	(junction
@@
 	(wire
 		(pts
-			(xy 162.56 95.25) (xy 171.45 95.25)
-		)
-		(stroke
-			(width 0)
-			(type default)
-		)
-	)
-	(wire
-		(pts
 			(xy 260.35 105.41) (xy 260.35 107.95)
 		)
@@
 	(wire
 		(pts
+			(xy 168.91 97.79) (xy 171.45 97.79)
+		)
+		(stroke
+			(width 0)
+			(type default)
+		)
+	)
+	(wire
+		(pts
 			(xy 237.49 107.95) (xy 245.11 107.95)
 		)
@@
 	(wire
 		(pts
+			(xy 171.45 95.25) (xy 171.45 90.17)
+		)
+		(stroke
+			(width 0)
+			(type default)
+		)
+	)
+	(wire
+		(pts
 			(xy 229.87 107.95) (xy 237.49 107.95)
 		)
@@
 	(wire
 		(pts
+			(xy 161.29 97.79) (xy 149.86 97.79)
+		)
+		(stroke
+			(width 0)
+			(type default)
+		)
+	)
+	(wire
+		(pts
 			(xy 220.98 130.81) (xy 207.01 130.81)
 		)
@@
 	(wire
 		(pts
+			(xy 149.86 97.79) (xy 149.86 96.52)
+		)
+		(stroke
+			(width 0)
+			(type default)
+		)
+	)
+	(wire
+		(pts
 			(xy 237.49 97.79) (xy 237.49 93.98)
 		)
@@
 	(wire
 		(pts
+			(xy 171.45 90.17) (xy 149.86 90.17)
+		)
+		(stroke
+			(width 0)
+			(type default)
+		)
+	)
+	(wire
+		(pts
 			(xy 245.11 107.95) (xy 252.73 107.95)
 		)
@@
 		(pts
 			(xy 220.98 114.3) (xy 220.98 130.81)
+		)
+		(stroke
+			(width 0)
+			(type default)
+		)
+	)
+	(wire
+		(pts
+			(xy 149.86 90.17) (xy 149.86 96.52)
 		)
 		(stroke
@@
 	(symbol
 		(lib_id "power:GND")
-		(at 162.56 95.25 270)
+		(at 149.86 96.52 270)
 		(unit 1)
 		(exclude_from_sim no)
@@
 		(dnp no)
 		(fields_autoplaced yes)
-		(property "Reference" "#PWR04"
-			(at 156.21 95.25 0)
+		(property "Reference" "#PWR06"
+			(at 143.51 96.52 0)
 			(effects
 				(font
@@
 		)
 		(property "Value" "GND"
-			(at 158.75 95.2499 90)
+			(at 146.05 96.5199 90)
 			(effects
 				(font
@@
 		)
 		(property "Footprint" ""
-			(at 162.56 95.25 0)
+			(at 149.86 96.52 0)
 			(effects
 				(font
@@
 		)
 		(property "Datasheet" ""
-			(at 162.56 95.25 0)
+			(at 149.86 96.52 0)
 			(effects
 				(font
@@
 		)
 		(property "Description" "Power symbol creates a global label with name \"GND\" , ground"
-			(at 162.56 95.25 0)
+			(at 149.86 96.52 0)
 			(effects
 				(font
@@
 		)
 		(instances
-			(project "LED_MATRIX"
+			(project ""
 				(path "/3e9d6c2e-f289-4b1b-ad37-c26dbc105080"
-					(reference "#PWR04")
+					(reference "#PWR06")
 					(unit 1)
 				)
@@
 					(unit 1)
 				)
+			)
+		)
+	)
+	(symbol
+		(lib_id "Device:R")
+		(at 165.1 97.79 90)
+		(unit 1)
+		(exclude_from_sim no)
+		(in_bom yes)
+		(on_board yes)
+		(dnp no)
+		(property "Reference" "R1"
+			(at 165.1 93.218 90)
+			(effects
+				(font
+					(size 1.27 1.27)
+				)
+			)
+		)
+		(property "Value" "2kO"
+			(at 165.1 95.758 90)
+			(effects
+				(font
+					(size 1.27 1.27)
+				)
+			)
+		)
+		(property "Footprint" ""
+			(at 165.1 99.568 90)
+			(effects
+				(font
+					(size 1.27 1.27)
+				)
+				(hide yes)
+			)
+		)
+		(property "Datasheet" "~"
+			(at 165.1 97.79 0)
+			(effects
+				(font
+					(size 1.27 1.27)
+				)
+				(hide yes)
+			)
+		)
+		(property "Description" "Resistor"
+			(at 165.1 97.79 0)
+			(effects
+				(font
+					(size 1.27 1.27)
+				)
+				(hide yes)
+			)
+		)
+		(pin "2"
+		)
+		(pin "1"
+		)
+		(instances
+			(project ""
+				(path "/3e9d6c2e-f289-4b1b-ad37-c26dbc105080"
+					(reference "R1")
+					(unit 1)
+				)

Commit message: Wip
Parts:
- added C1: C_Polarized_US, symbol Device:C_Polarized_US
- added C2: C, symbol Device:C
Connections:
- net GND: now also C1.2, C2.2
- net VCC: now also C1.1, C2.1

Commit message: wip
Parts:
- C1: value C_Polarized_US -> 4.7uF; footprint (none) -> Capacitor_SMD:C_0504_1310Metric_Pad0.83x1.28mm_HandSolder
- C2: value C -> 0.1uF; footprint (none) -> Capacitor_SMD:C_0504_1310Metric_Pad0.83x1.28mm_HandSolder
- R1: footprint (none) -> Resistor_SMD:R_1206_3216Metric_Pad1.30x1.75mm_HandSolder
- TP1, TP2, TP3, TP4, TP5: footprint TestPoint:TestPoint_Pad_1.5x1.5mm -> TestPoint:TestPoint_Pad_1.0x1.0mm
Connections:
- net GND: now also U2.29 (PAD)
Changed lines of the file:
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@@
+	(wire
+		(pts
+			(xy 186.69 140.97) (xy 186.69 146.05)
+		)
+		(stroke
+			(width 0)
+			(type default)
+		)
+	)
 	(wire
 		(pts
 			(xy 260.35 118.11) (xy 260.35 110.49)
+		)
+		(stroke
+			(width 0)
+			(type default)
+		)
+	)
+	(wire
+		(pts
+			(xy 186.69 146.05) (xy 189.23 146.05)
 		)
 		(stroke
@@
 			)
 		)
-		(property "Value" "C_Polarized_US"
+		(property "Value" "4.7uF"
 			(at 232.41 150.4949 0)
 			(effects
@@
 			)
 		)
-		(property "Footprint" ""
+		(property "Footprint" "Capacitor_SMD:C_0504_1310Metric_Pad0.83x1.28mm_HandSolder"
 			(at 228.6 149.86 0)
 			(effects
@@
 			)
 		)
-		(property "Value" "C"
+		(property "Value" "0.1uF"
 			(at 219.71 151.1299 0)
 			(effects
@@
 			)
 		)
-		(property "Footprint" ""
+		(property "Footprint" "Capacitor_SMD:C_0504_1310Metric_Pad0.83x1.28mm_HandSolder"
 			(at 216.8652 153.67 0)
 			(effects
@@
 			)
 		)
-		(property "Footprint" ""
+		(property "Footprint" "Resistor_SMD:R_1206_3216Metric_Pad1.30x1.75mm_HandSolder"
 			(at 165.1 99.568 90)
 			(effects
@@
 			)
 		)
-		(property "Footprint" "TestPoint:TestPoint_Pad_1.5x1.5mm"
+		(property "Footprint" "TestPoint:TestPoint_Pad_1.0x1.0mm"
 			(at 162.56 123.19 0)
 			(effects
@@
 			)
 		)
-		(property "Footprint" "TestPoint:TestPoint_Pad_1.5x1.5mm"
+		(property "Footprint" "TestPoint:TestPoint_Pad_1.0x1.0mm"
 			(at 162.56 102.87 0)
 			(effects
@@
 			)
 		)
-		(property "Footprint" "TestPoint:TestPoint_Pad_1.5x1.5mm"
+		(property "Footprint" "TestPoint:TestPoint_Pad_1.0x1.0mm"
 			(at 162.56 125.73 0)
 			(effects
@@
 			)
 		)
-		(property "Footprint" "TestPoint:TestPoint_Pad_1.5x1.5mm"
+		(property "Footprint" "TestPoint:TestPoint_Pad_1.0x1.0mm"
 			(at 162.56 105.41 0)
 			(effects
@@
 			)
 		)
-		(property "Footprint" "TestPoint:TestPoint_Pad_1.5x1.5mm"
+		(property "Footprint" "TestPoint:TestPoint_Pad_1.0x1.0mm"
 			(at 162.56 97.79 0)
 			(effects

Commit message: wip
Parts:
- added TP6, TP7: TestPoint, TestPoint:TestPoint_Pad_1.0x1.0mm, symbol Connector:TestPoint
- U2: footprint Package_SO:HTSSOP-28-1EP_4.4x9.7mm_P0.65mm_EP3.4x9.5mm_Mask2.4x6.17mm_ThermalVias -> Footprints:HTSSOP-28-1EP_4.4x9.7mm_P0.65mm_EP3.4x9.5mm_Mask2.4x6.17mm_ThermalVias_OnlyFrontCopper
Connections:
- net GND: now also TP7.1
- net VCC: now also TP6.1
