File: LED_MATRIX.kicad_pcb (KiCad board)
At the start: 2 copper layers, 16 parts, among them J1 Conn_01x01, J2 Conn_01x01, U1 AS1115-BSST

Commit message: wip
Parts:
- removed J1, J2: Conn_01x01, TestPoint:TestPoint_THTPad_2.0x2.0mm_Drill1.0mm
- removed U1: AS1115-BSST, Package_SO:QSOP-24_3.9x8.7mm_P0.635mm
- added C1: 4.7uF, Capacitor_SMD:C_0504_1310Metric_Pad0.83x1.28mm_HandSolder, F.Cu at (246.8, 156.6)
- added C2: 0.1uF, Capacitor_SMD:C_0504_1310Metric_Pad0.83x1.28mm_HandSolder, F.Cu at (248.4, 156.6)
- added TP1: TestPoint, TestPoint:TestPoint_Pad_1.0x1.0mm, F.Cu at (241.4, 151.5)
- added TP2: TestPoint, TestPoint:TestPoint_Pad_1.0x1.0mm, F.Cu at (243.4, 151.5)
- added TP3: TestPoint, TestPoint:TestPoint_Pad_1.0x1.0mm, F.Cu at (245.4, 151.5)
- added TP4: TestPoint, TestPoint:TestPoint_Pad_1.0x1.0mm, F.Cu at (241.4, 153.5)
- added TP5: TestPoint, TestPoint:TestPoint_Pad_1.0x1.0mm, F.Cu at (243.4, 153.5)
- added U2: TLC5940PWP, Package_SO:HTSSOP-28-1EP_4.4x9.7mm_P0.65mm_EP3.4x9.5mm_Mask2.4x6.17mm_ThermalVias, F.Cu at (235.3, 154.1)
- D1: moved to B.Cu
- R1: value 9.53kOhm -> 2kO; footprint Resistor_SMD:R_0805_2012Metric_Pad1.20x1.40mm_HandSolder -> Resistor_SMD:R_1206_3216Metric_Pad1.30x1.75mm_HandSolder; moved to F.Cu
- moved D1 91.7 mm to (247.5, 155.2)
- moved R1 78.4 mm to (248.2, 152.9), turned to -90 degrees
- moved D3 71.9 mm to (249.8, 143.2)
- moved D8 71.9 mm to (236.3, 143.2)
- moved D10 71.9 mm to (230.9, 143.2)
- moved D11 71.9 mm to (228.2, 143.2)
- moved D12 71.9 mm to (225.5, 143.2)
- moved D4 71.9 mm to (247.1, 143.2)
- moved D5 71.9 mm to (244.4, 143.2)
- moved D6 71.9 mm to (241.7, 143.2)
- moved D7 71.9 mm to (239.0, 143.2)
- moved D9 71.9 mm to (233.6, 143.2)
- moved D2 65.9 mm to (243.0, 155.2), turned to 0 degrees
Connections:
- D1 pad 2: Net-(D1-A) -> VCC
- D10 pad 2: Net-(D10-A) -> VCC
- D11 pad 2: Net-(D1-A) -> VCC
- D12 pad 1: Net-(D11-K) -> Net-(D12-K)
- D12 pad 2: Net-(D10-A) -> VCC
- D2 pad 1: Net-(D1-K) -> Net-(D2-K)
- D2 pad 2: Net-(D2-A) -> VCC
- D3 pad 1: Net-(D1-K) -> Net-(D3-K)
- D3 pad 2: Net-(D3-A) -> VCC
- D4 pad 1: Net-(D1-K) -> Net-(D4-K)
- D4 pad 2: Net-(D4-A) -> VCC
- D5 pad 1: Net-(D1-K) -> Net-(D5-K)
- D5 pad 2: Net-(D10-A) -> VCC
- D6 pad 1: Net-(D10-K) -> Net-(D6-K)
- D6 pad 2: Net-(D1-A) -> VCC
- D7 pad 1: Net-(D10-K) -> Net-(D7-K)
- D7 pad 2: Net-(D2-A) -> VCC
- D8 pad 1: Net-(D10-K) -> Net-(D8-K)
- D8 pad 2: Net-(D3-A) -> VCC
- D9 pad 1: Net-(D10-K) -> Net-(D9-K)
- D9 pad 2: Net-(D4-A) -> VCC
- R1 pad 1: VCC -> GND

Commit message: wip
Parts:
- added TP6: TestPoint, TestPoint:TestPoint_Pad_1.0x1.0mm, B.Cu at (264.0, 147.8)
- added TP7: TestPoint, TestPoint:TestPoint_Pad_1.0x1.0mm, B.Cu at (262.0, 147.8)
- C1, C2, R1, TP1, TP2, TP3, TP4, TP5: moved to B.Cu
- D1, D10, D11, D12, D2, D3, D4, D5, D6, D7, D8, D9: moved to F.Cu
- U2: footprint Package_SO:HTSSOP-28-1EP_4.4x9.7mm_P0.65mm_EP3.4x9.5mm_Mask2.4x6.17mm_ThermalVias -> Footprints:HTSSOP-28-1EP_4.4x9.7mm_P0.65mm_EP3.4x9.5mm_Mask2.4x6.17mm_ThermalVias_OnlyFrontCopper; moved to B.Cu
- moved D12 46.0 mm to (270.8, 151.8), turned to 0 degrees
- moved D10 44.9 mm to (275.8, 145.5), turned to 0 degrees
- moved D9 43.0 mm to (275.8, 151.8), turned to 0 degrees
- moved D8 42.2 mm to (275.8, 158.2)
- moved U2 35.4 mm to (270.2, 148.4)
- moved D7 35.1 mm to (270.8, 158.2)
- moved D6 28.3 mm to (265.8, 158.2)
- moved D11 27.6 mm to (255.8, 145.5), turned to 0 degrees
- moved D5 22.2 mm to (260.8, 158.2)
- moved TP4 22.0 mm to (262.0, 145.8), turned to 180 degrees
- moved TP2 21.3 mm to (264.0, 145.8), turned to 180 degrees
- moved TP1 19.4 mm to (260.0, 145.8), turned to 180 degrees
- moved D2 18.1 mm to (260.8, 151.8)
- moved D3 18.1 mm to (265.8, 151.8), turned to 0 degrees
- moved D4 17.3 mm to (255.8, 158.2)
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Routing:
- net VCC: track 0.00 -> 97.7 mm, vias 0 -> 1
- net Net-(D11-K): track 0.00 -> 26.3 mm, vias 0 -> 1
- net GND: track 0.00 -> 22.7 mm
- net Net-(D4-K): track 0.00 -> 18.7 mm, vias 0 -> 1
- net Net-(D1-K): track 0.00 -> 15.5 mm, vias 0 -> 1
- net Net-(D5-K): track 0.00 -> 14.3 mm, vias 0 -> 1
- net Net-(U2-SIN): track 0.00 -> 12.4 mm
- net Net-(D2-K): track 0.00 -> 11.1 mm, vias 0 -> 1
- net Net-(D3-K): track 0.00 -> 11.0 mm, vias 0 -> 1
- net Net-(U2-GSCLK): track 0.00 -> 10.5 mm
- net Net-(D9-K): track 0.00 -> 10.4 mm, vias 0 -> 2
- net Net-(D6-K): track 0.00 -> 9.97 mm, vias 0 -> 1
- net Net-(U2-SCLK): track 0.00 -> 9.51 mm
- net Net-(D12-K): track 0.00 -> 8.67 mm, vias 0 -> 1
- net Net-(U2-XLAT): track 0.00 -> 7.13 mm
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- added copper zone on B.Cu, net GND
- added copper zone on F.Cu, net GND
Other:
- board outline added: 23.5 x 19 mm
- copper layers 2 -> 4
