File: LedMatrix.kicad_pcb (KiCad board)
At the start: 4 copper layers, 24 x 13 mm, 23 parts, among them U2 TLC5940PWP

Commit message: 2.1
Parts:
- moved 2 4.47 mm to (198.8, 160.0)
- moved 5 0.98 mm to (196.8, 160.0)
Routing:
- net GND: track 11.8 -> 27.2 mm
- net Net-(U2-BLANK): track 22.1 -> 36.7 mm, vias 0 -> 2
- net Net-(U2-GSCLK): track 10.9 -> 13.8 mm
- net Net-(D6-K): track 8.90 -> 11.6 mm
- net Net-(D1-K): track 11.3 -> 13.1 mm
- net VCC: track 72.1 -> 70.4 mm
- net Net-(D7-K): track 7.79 -> 6.50 mm
- net Net-(D10-K): track 9.05 -> 7.85 mm
- net Net-(D5-K): track 5.11 -> 5.81 mm
- net Net-(D2-K): track 7.31 -> 7.91 mm

Commit message: 2.3
Parts:
- D1, D10, D11, D12, D2, D3, D4, D5, D6, D7, D8, D9: footprint Footprints:Bivar_1206_SMD -> Footprints:SM1206UWCIL
- renumbered 2 to BLNK, G to GND, 5 to GSCLK, 1 to SCLK, 3 to SIN, V to VCC, 4 to XLAT
Routing:
- net VCC: track 70.4 -> 68.0 mm
- net Net-(D6-K): track 11.6 -> 9.98 mm
- net Net-(U2-BLANK): track 36.7 -> 35.9 mm
- net Net-(D5-K): track 5.81 -> 5.11 mm

Commit message: 2.4
Parts:
- C1, C2: footprint Capacitor_SMD:C_0504_1310Metric_Pad0.83x1.28mm_HandSolder -> Footprints:C_0504_1310Metric_Pad0.83x1.28mm_HandSolder
Changed lines of the file:
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@@
 		(embedded_fonts no)
 	)
-	(footprint "Capacitor_SMD:C_0504_1310Metric_Pad0.83x1.28mm_HandSolder"
+	(footprint "Footprints:C_0504_1310Metric_Pad0.83x1.28mm_HandSolder"
 		(layer "B.Cu")
 		(at 183.97 157.5275 90)
@@
 		(tags "capacitor handsolder")
 		(property "Reference" "C1"
-			(at 1.6225 0 0)
+			(at 1.7775 0.03 180)
 			(layer "B.SilkS")
 			(effects
@@
 		)
 		(property "Value" "4.7uF"
-			(at 0 -1.49 90)
+			(at 0 -1.49 270)
 			(layer "B.Fab")
 			(effects
@@
 		)
 		(property "Datasheet" "~"
-			(at 0 0 90)
+			(at 0 0 270)
 			(layer "B.Fab")
 			(hide yes)
@@
 		)
 		(property "Description" "Polarized capacitor, US symbol"
-			(at 0 0 90)
+			(at 0 0 270)
 			(layer "B.Fab")
 			(hide yes)
@@
 		)
 		(fp_text user "${REFERENCE}"
-			(at 0 0 90)
+			(at 0 0 270)
 			(layer "B.Fab")
 			(effects
@@
 		)
 		(embedded_fonts no)
-		(model "${KICAD9_3DMODEL_DIR}/Capacitor_SMD.3dshapes/C_0504_1310Metric.step"
+		(model "${KIPRJMOD}/3DModels/0504B103J101PT.stp"
 			(offset
 				(xyz 0 0 0)
@@
 		(tags "TSSOP HTSSOP 0.65 thermal pad")
 		(property "Reference" "U2"
-			(at 0 3.75 90)
+			(at -4.65 0.22 0)
 			(layer "B.SilkS")
 			(effects
@@
 		)
 	)
-	(footprint "Capacitor_SMD:C_0504_1310Metric_Pad0.83x1.28mm_HandSolder"
+	(footprint "Footprints:C_0504_1310Metric_Pad0.83x1.28mm_HandSolder"
 		(layer "B.Cu")
 		(at 181.5975 160.15 180)
@@
 		)
 		(embedded_fonts no)
-		(model "${KICAD9_3DMODEL_DIR}/Capacitor_SMD.3dshapes/C_0504_1310Metric.step"
+		(model "${KIPRJMOD}/3DModels/0504B103J101PT.stp"
 			(offset
 				(xyz 0 0 0)
@@
 		(tags "test point SMD pad rectangle square")
 		(property "Reference" "GND"
-			(at 0 1.9 0)
+			(at -0.03 1.65 0)
 			(layer "B.SilkS")
 			(effects
@@
 		(tags "test point SMD pad rectangle square")
 		(property "Reference" "VCC"
-			(at 0 -2.1 0)
-			(layer "B.SilkS")
-			(effects
+			(at 0 -1.85 0)
+			(layer "B.SilkS")
+			(effects
