File: LedMatrix.kicad_pcb (KiCad board)
At the start: 4 copper layers, 24 x 13 mm, 23 parts, among them U2 TLC5940PWP

Commit message: 2.5
Parts:
- added C3: 4.7uF, Footprints:C_0504_1310Metric_Pad0.83x1.28mm_HandSolder, B.Cu at (181.6, 158.5)
Routing:
- net GND: track 27.2 -> 31.6 mm
- net VCC: track 68.0 -> 69.5 mm
Other:
- board text added: "v2.5"

Commit message: 2.6
Other:
- board text added: "v${REVISION}"
- board text removed: "v2.5"
Changed lines of the file:
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@@
 		(title "LedMatrix PCB")
 		(date "2025-11-16")
-		(rev "2.5")
+		(rev "2.6")
 		(company "HAW Hamburg")
 	)
@@
 		(layer "Edge.Cuts")
 	)
-	(gr_text "v2.5"
+	(gr_text "v${REVISION}"
 		(at 200.75 160 270)
 		(layer "B.SilkS")
@@
 		(start 181.47 157.72)
 		(end 181.47 155.673)
-		(width 0.127)
+		(width 0.2)
 		(layer "F.Cu")
 		(net 11)
@@
 		(start 188.12 157.9)
 		(end 192.32 157.9)
-		(width 0.127)
+		(width 0.2)
 		(layer "F.Cu")
 		(net 11)
@@
 		(start 188.12 151.4)
 		(end 192.32 151.4)
-		(width 0.127)
-		(layer "F.Cu")
-		(net 11)
-	)
-	(segment
-		(start 192.32 159.243084)
-		(end 192.32 157.9)
-		(width 0.127)
+		(width 0.2)
 		(layer "F.Cu")
 		(net 11)
@@
 		(start 200.57 157.9)
 		(end 196.52 157.9)
-		(width 0.127)
+		(width 0.2)
 		(layer "F.Cu")
 		(net 11)
@@
 		(start 196.67 151.25)
 		(end 196.52 151.4)
-		(width 0.127)
-		(layer "F.Cu")
-		(net 11)
-	)
-	(segment
-		(start 196.52 158.096088)
-		(end 194.124588 160.4915)
-		(width 0.127)
+		(width 0.2)
 		(layer "F.Cu")
 		(net 11)
@@
 		(start 179.9 157.72)
 		(end 179.72 157.9)
-		(width 0.127)
+		(width 0.2)
 		(layer "F.Cu")
 		(net 11)
@@
 		(start 181.75 151.5)
 		(end 181.85 151.4)
-		(width 0.127)
+		(width 0.2)
 		(layer "F.Cu")
 		(net 11)
@@
 		(start 181.65 151.4)
 		(end 179.72 151.4)
-		(width 0.127)
+		(width 0.2)
 		(layer "F.Cu")
 		(net 11)
@@
 		(start 182.65 158.9)
 		(end 181.47 157.72)
-		(width 0.127)
+		(width 0.2)
 		(layer "F.Cu")
 		(net 11)
@@
 		(start 201.354193 157.115807)
 		(end 200.57 157.9)
-		(width 0.127)
+		(width 0.2)
 		(layer "F.Cu")
 		(net 11)
@@
 		(start 201.354193 156.077002)
 		(end 201.354193 157.265807)
-		(width 0.127)
+		(width 0.2)
+		(layer "F.Cu")
+		(net 11)
+	)
+	(segment
+		(start 194.2 160.7)
+		(end 193.6 160.7)
+		(width 0.2)
 		(layer "F.Cu")
 		(net 11)
@@
 		(start 200.72 151.4)
 		(end 200.57 151.25)
-		(width 0.127)
+		(width 0.2)
+		(layer "F.Cu")
+		(net 11)
+	)
+	(segment
+		(start 193.6 160.7)
+		(end 192.32 159.42)
+		(width 0.2)
 		(layer "F.Cu")
 		(net 11)
@@
 		(start 183.92 151.4)
 		(end 188.12 151.4)
-		(width 0.127)
+		(width 0.2)
 		(layer "F.Cu")
 		(net 11)
@@
 		(start 183.92 157.9)
 		(end 188.12 157.9)
-		(width 0.127)
+		(width 0.2)
 		(layer "F.Cu")
 		(net 11)
@@
 		(start 183.97 159.9)
 		(end 182.97 158.9)
-		(width 0.127)
+		(width 0.2)
 		(layer "F.Cu")
 		(net 11)
 	)
 	(segment
-		(start 194.124588 160.4915)
-		(end 193.568416 160.4915)
-		(width 0.127)
+		(start 182.97 158.9)
+		(end 182.65 158.9)
+		(width 0.2)
 		(layer "F.Cu")
 		(net 11)
 	)
 	(segment
-		(start 182.97 158.9)
-		(end 182.65 158.9)
-		(width 0.127)
+		(start 201.354193 156.077002)
+		(end 201.354193 157.115807)
+		(width 0.2)
 		(layer "F.Cu")
 		(net 11)
 	)
 	(segment
-		(start 201.354193 157.265807)
-		(end 200.72 157.9)
-		(width 0.127)
+		(start 196.52 157.9)
+		(end 196.52 158.38)
+		(width 0.2)
 		(layer "F.Cu")
 		(net 11)
 	)
 	(segment
-		(start 201.354193 156.077002)
-		(end 201.354193 157.115807)
-		(width 0.127)
+		(start 196.52 158.38)
+		(end 194.2 160.7)
+		(width 0.2)
 		(layer "F.Cu")
 		(net 11)
@@
 		(start 182.97 158.9)
 		(end 182.97 158.85)
-		(width 0.127)
+		(width 0.2)
 		(layer "F.Cu")
 		(net 11)
@@
 		(start 181.75 151.5)
 		(end 181.65 151.4)
-		(width 0.127)
+		(width 0.2)
 		(layer "F.Cu")
 		(net 11)
 	)
 	(segment
-		(start 200.57 151.25)
-		(end 196.67 151.25)
-		(width 0.127)
+		(start 192.32 159.42)
+		(end 192.32 157.9)
+		(width 0.2)
 		(layer "F.Cu")
 		(net 11)
 	)
 	(segment
-		(start 193.568416 160.4915)
-		(end 192.32 159.243084)
-		(width 0.127)
+		(start 200.57 151.25)
+		(end 196.67 151.25)
+		(width 0.2)
 		(layer "F.Cu")
 		(net 11)
@@
 		(start 181.47 157.72)
 		(end 179.9 157.72)
-		(width 0.127)
-		(layer "F.Cu")
-		(net 11)
-	)
-	(segment
-		(start 196.52 157.9)
-		(end 196.52 158.096088)
-		(width 0.127)
+		(width 0.2)
 		(layer "F.Cu")
 		(net 11)
@@
 		(start 181.85 151.4)
 		(end 183.92 151.4)
-		(width 0.127)
+		(width 0.2)
 		(layer "F.Cu")
 		(net 11)
@@
 		(start 182.97 158.85)
 		(end 183.92 157.9)
-		(width 0.127)
+		(width 0.2)
 		(layer "F.Cu")
 		(net 11)
@@
 	)
 	(segment
-		(start 182.7865 152.5365)
-		(end 181.75 151.5)
-		(width 0.127)
+		(start 185.995 159.75)
+		(end 185.995 159.073)
+		(width 0.2)
 		(layer "B.Cu")
 		(net 11)
 	)
 	(segment
-		(start 187.295 159.267)
-		(end 187.295 159.75)
-		(width 0.127)
+		(start 183.97 159.9)
+		(end 183.97 158.155)
+		(width 0.2)
 		(layer "B.Cu")
 		(net 11)
 	)
 	(segment
-		(start 183.97 159.9)
-		(end 183.97 158.155)
-		(width 0.127)
+		(start 186.928 158.9)
+		(end 187.295 159.267)
+		(width 0.2)
 		(layer "B.Cu")
 		(net 11)
@@
 		(start 183.97 159.9)
 		(end 185.845 159.9)
-		(width 0.127)
+		(width 0.2)
 		(layer "B.Cu")
 		(net 11)
@@
 		(start 200.72 155.442809)
 		(end 200.72 151.4)
-		(width 0.127)
+		(width 0.2)
 		(layer "B.Cu")
 		(net 11)
@@
 		(start 182.475 159.9)
 		(end 182.225 160.15)
-		(width 0.127)
+		(width 0.2)
 		(layer "B.Cu")
 		(net 11)
 	)
 	(segment
-		(start 182.7865 154.3565)
-		(end 182.7865 152.5365)
-		(width 0.127)
+		(start 182.225 160.15)
+		(end 182.225 159.005624)
+		(width 0.2)
 		(layer "B.Cu")
 		(net 11)
 	)
 	(segment
-		(start 182.225 160.15)
-		(end 182.225 159.005624)
-		(width 0.127)
+		(start 183 152.75)
+		(end 181.75 151.5)
+		(width 0.2)
 		(layer "B.Cu")
 		(net 11)
@@
 		(start 183.97 159.9)
 		(end 182.475 159.9)
-		(width 0.127)
+		(width 0.2)
 		(layer "B.Cu")
 		(net 11)
 	)
 	(segment
-		(start 186.0595 159.0085)
-		(end 187.0365 159.0085)
-		(width 0.127)
+		(start 186.168 158.9)
+		(end 186.928 158.9)
+		(width 0.2)
 		(layer "B.Cu")
 		(net 11)
 	)
 	(segment
-		(start 181.47 155.673)
-		(end 182.7865 154.3565)
-		(width 0.127)
+		(start 201.354193 156.077002)
+		(end 200.72 155.442809)
+		(width 0.2)
 		(layer "B.Cu")
 		(net 11)
 	)
 	(segment
-		(start 185.995 159.073)
-		(end 186.0595 159.0085)
-		(width 0.127)
+		(start 185.845 159.9)
+		(end 185.995 159.75)
+		(width 0.2)
 		(layer "B.Cu")
 		(net 11)
 	)
 	(segment
-		(start 185.995 159.75)
-		(end 185.995 159.073)
-		(width 0.127)
+		(start 187.295 159.267)
+		(end 187.295 159.75)
+		(width 0.2)
 		(layer "B.Cu")
 		(net 11)
 	)
 	(segment
-		(start 201.354193 156.077002)
-		(end 200.72 155.442809)
-		(width 0.127)
+		(start 185.995 159.073)
+		(end 186.168 158.9)
+		(width 0.2)
 		(layer "B.Cu")
 		(net 11)
 	)
 	(segment
-		(start 185.845 159.9)
-		(end 185.995 159.75)
-		(width 0.127)
+		(start 183 154.143)
+		(end 183 152.75)
+		(width 0.2)
 		(layer "B.Cu")
 		(net 11)
@@
 		(start 182.225 159.005624)
 		(end 182.490312 158.740312)
-		(width 0.127)
+		(width 0.2)
 		(layer "B.Cu")
 		(net 11)
 	)
 	(segment
-		(start 187.0365 159.0085)
-		(end 187.295 159.267)
-		(width 0.127)
+		(start 181.47 155.673)
+		(end 183 154.143)
+		(width 0.2)
 		(layer "B.Cu")
 		(net 11)
@@
 		(layers "F.Cu" "B.Cu")
 		(hatch edge 0.5)
-		(connect_pads
+		(connect_pads yes
 			(clearance 0.5)
 		)
