File: LedMatrix.kicad_sch (KiCad schematic)
At the start: 23 parts, among them U2 TLC5940PWP

Commit message: 2.3
Parts:
- D1, D10, D11, D12, D2, D3, D4, D5, D6, D7, D8, D9: footprint Footprints:Bivar_1206_SMD -> Footprints:SM1206UWCIL
Changed lines of the file:
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@@
 			)
 		)
-		(property "Footprint" "Footprints:Bivar_1206_SMD"
+		(property "Footprint" "Footprints:SM1206UWCIL"
 			(at 245.11 101.6 0)
 			(effects
@@
 			)
 		)
-		(property "Footprint" "Footprints:Bivar_1206_SMD"
+		(property "Footprint" "Footprints:SM1206UWCIL"
 			(at 260.35 80.01 0)
 			(effects
@@
 			)
 		)
-		(property "Footprint" "Footprints:Bivar_1206_SMD"
+		(property "Footprint" "Footprints:SM1206UWCIL"
 			(at 260.35 101.6 0)
 			(effects
@@
 			)
 		)
-		(property "Footprint" "Footprints:Bivar_1206_SMD"
+		(property "Footprint" "Footprints:SM1206UWCIL"
 			(at 229.87 80.01 0)
 			(effects
@@
 			)
 		)
-		(property "Footprint" "Footprints:Bivar_1206_SMD"
+		(property "Footprint" "Footprints:SM1206UWCIL"
 			(at 252.73 121.92 0)
 			(effects
@@
 			)
 		)
-		(property "Footprint" "Footprints:Bivar_1206_SMD"
+		(property "Footprint" "Footprints:SM1206UWCIL"
 			(at 237.49 101.6 0)
 			(effects
@@
 			)
 		)
-		(property "Footprint" "Footprints:Bivar_1206_SMD"
+		(property "Footprint" "Footprints:SM1206UWCIL"
 			(at 245.11 121.92 0)
 			(effects
@@
 			)
 		)
-		(property "Footprint" "Footprints:Bivar_1206_SMD"
+		(property "Footprint" "Footprints:SM1206UWCIL"
 			(at 252.73 101.6 0)
 			(effects
@@
 			)
 		)
-		(property "Footprint" "Footprints:Bivar_1206_SMD"
+		(property "Footprint" "Footprints:SM1206UWCIL"
 			(at 229.87 101.6 0)
 			(effects
@@
 			)
 		)
-		(property "Footprint" "Footprints:Bivar_1206_SMD"
+		(property "Footprint" "Footprints:SM1206UWCIL"
 			(at 237.49 121.92 0)
 			(effects
@@
 			)
 		)
-		(property "Footprint" "Footprints:Bivar_1206_SMD"
+		(property "Footprint" "Footprints:SM1206UWCIL"
 			(at 260.35 121.92 0)
 			(effects
@@
 			)
 		)
-		(property "Footprint" "Footprints:Bivar_1206_SMD"
+		(property "Footprint" "Footprints:SM1206UWCIL"
 			(at 229.87 121.92 0)
 			(effects

Commit message: 2.4
Parts:
- C1, C2: footprint Capacitor_SMD:C_0504_1310Metric_Pad0.83x1.28mm_HandSolder -> Footprints:C_0504_1310Metric_Pad0.83x1.28mm_HandSolder
Changed lines of the file:
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@@
 			)
 		)
-		(property "Footprint" "Capacitor_SMD:C_0504_1310Metric_Pad0.83x1.28mm_HandSolder"
+		(property "Footprint" "Footprints:C_0504_1310Metric_Pad0.83x1.28mm_HandSolder"
 			(at 228.6 149.86 0)
 			(effects
@@
 			)
 		)
-		(property "Footprint" "Capacitor_SMD:C_0504_1310Metric_Pad0.83x1.28mm_HandSolder"
+		(property "Footprint" "Footprints:C_0504_1310Metric_Pad0.83x1.28mm_HandSolder"
 			(at 216.8652 153.67 0)
 			(effects

Commit message: 2.5
Parts:
- added C3: 4.7uF, Footprints:C_0504_1310Metric_Pad0.83x1.28mm_HandSolder, symbol Device:C_Polarized_US
Connections:
- net GND: now also C3.2
- net VCC: now also C3.1
Changed lines of the file:
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@@
+	)
+	(junction
+		(at 241.3 142.24)
+		(diameter 0)
+		(color 0 0 0 0)
 	)
 	(junction
@@
 	)
 	(junction
+		(at 228.6 157.48)
+		(diameter 0)
+		(color 0 0 0 0)
+	)
+	(junction
 		(at 260.35 86.36)
 		(diameter 0)
@@
 	(wire
 		(pts
+			(xy 241.3 142.24) (xy 241.3 146.05)
+		)
+		(stroke
+			(width 0)
+			(type default)
+		)
+	)
+	(wire
+		(pts
 			(xy 252.73 111.76) (xy 218.44 111.76)
 		)
@@
 	(wire
 		(pts
+			(xy 228.6 157.48) (xy 241.3 157.48)
+		)
+		(stroke
+			(width 0)
+			(type default)
+		)
+	)
+	(wire
+		(pts
 			(xy 229.87 115.57) (xy 222.25 115.57)
 		)
@@
 	(wire
 		(pts
-			(xy 228.6 142.24) (xy 273.05 142.24)
+			(xy 241.3 157.48) (xy 241.3 153.67)
+		)
+		(stroke
+			(width 0)
+			(type default)
+		)
+	)
+	(wire
+		(pts
+			(xy 228.6 142.24) (xy 241.3 142.24)
 		)
 		(stroke
@@
 		(pts
 			(xy 228.6 142.24) (xy 228.6 146.05)
+		)
+		(stroke
+			(width 0)
+			(type default)
+		)
+	)
+	(wire
+		(pts
+			(xy 241.3 142.24) (xy 273.05 142.24)
 		)
 		(stroke
@@
 					(unit 1)
 				)
+			)
+		)
+	)
+	(symbol
+		(lib_id "Device:C_Polarized_US")
+		(at 241.3 149.86 0)
+		(unit 1)
+		(exclude_from_sim no)
+		(in_bom yes)
+		(on_board yes)
+		(dnp no)
+		(fields_autoplaced yes)
+		(property "Reference" "C3"
+			(at 245.11 147.9549 0)
+			(effects
+				(font
+					(size 1.27 1.27)
+				)
+				(justify left)
+			)
+		)
+		(property "Value" "4.7uF"
+			(at 245.11 150.4949 0)
+			(effects
+				(font
+					(size 1.27 1.27)
+				)
+				(justify left)
+			)
+		)
+		(property "Footprint" "Footprints:C_0504_1310Metric_Pad0.83x1.28mm_HandSolder"
+			(at 241.3 149.86 0)
+			(effects
+				(font
+					(size 1.27 1.27)
+				)
+				(hide yes)
+			)
+		)
+		(property "Datasheet" "~"
+			(at 241.3 149.86 0)
+			(effects
+				(font
+					(size 1.27 1.27)
+				)
+				(hide yes)
+			)
+		)
+		(property "Description" "Polarized capacitor, US symbol"
+			(at 241.3 149.86 0)
+			(effects
+				(font
+					(size 1.27 1.27)
+				)
+				(hide yes)
+			)
+		)
+		(pin "1"
+		)
+		(pin "2"
+		)
+		(instances
+			(project "LedMatrix"
+				(path "/3e9d6c2e-f289-4b1b-ad37-c26dbc105080"
+					(reference "C3")
+					(unit 1)
+				)
